Commit message: completed the 6th link of the brilliance called XARM7

File: urdf/arm7.urdf (robot description, URDF)
Before this commit: robot Xarm7, 4 links, 3 joints
Links:
- added link link3; visual mesh filename=package://xarm7_description/meshes/link3.stl scale=1.0 1.0 1.0
- added link link4; visual mesh filename=package://xarm7_description/meshes/link4.stl scale=1.0 1.0 1.0
- added link link5; visual mesh filename=package://xarm7_description/meshes/link5.stl scale=1.0 1.0 1.0
- added link link6; visual mesh filename=package://xarm7_description/meshes/link6.stl scale=1.0 1.0 1.0
Joints:
- added joint link2-link3: type revolute, parent link2, child link3, origin xyz=0 0.0 0.291 rpy=0 0.0 0.0, axis 0.0 0 1, limit lower=-3.14 upper=3.14 effort=0.0 velocity=0.0
- added joint link3-link4: type revolute, parent link3, child link4, origin xyz=0.057 0 0 rpy=0 0.0 0.0, axis 0.0 1 0, limit lower=-3.140 upper=3.140 effort=0.0 velocity=0.0
- added joint link4-link5: type revolute, parent link4, child link5, origin xyz=0.0782 0 -0.342 rpy=0 0.0 0.0, axis 0 0 1, limit lower=-3.140 upper=3.140 effort=0.0 velocity=0.0
- added joint link5-link6: type revolute, parent link5, child link6, origin xyz=0.0022 0 0.0045 rpy=0 0 0.0, axis 0 1 0, limit lower=-3.140 upper=3.140 effort=0.0 velocity=0.0
- joint base_link-link1: origin xyz=0.0 0.0 0.043 rpy=0.0 0.0 0.0 -> xyz=0.0 0.0 0.037 rpy=0.0 0.0 0.0
- joint link1-link2: limit lower=-3.14 upper=3.14 effort=0.0 velocity=0.0 -> lower=-2.0 upper=2.0 effort=0.0 velocity=0.0; origin xyz=0.15 0.16 0.23 rpy=0.0 0.0 0.0 -> xyz=0 0.0 0.23 rpy=0 0.0 0.0

Commit message: finalizaion of the XARM7 arm

File: urdf/arm7.urdf (robot description, URDF)
Before this commit: robot Xarm7, 8 links, 7 joints
Links:
- added link gripper; visual mesh filename=package://xarm7_description/meshes/gripper_lite.stl scale=1.0 1.0 1.0
- added link link7; visual mesh filename=package://xarm7_description/meshes/link7.stl scale=1.0 1.0 1.0
Joints:
- added joint link6-link7: type revolute, parent link6, child link7, origin xyz=0.076 0 -0.069 rpy=0 0.0 0.0, axis 0 0 1, limit lower=-3.140 upper=3.140 effort=0.0 velocity=0.0
- added joint link7-gripper: type fixed, parent link7, child gripper, origin xyz=0.0 0 -0.028 rpy=0 0.0 0.0
- joint link2-link3: limit lower=-3.14 upper=3.14 effort=0.0 velocity=0.0 -> lower=-2.2 upper=2.2 effort=0.0 velocity=0.0
- joint link3-link4: limit lower=-3.140 upper=3.140 effort=0.0 velocity=0.0 -> lower=-4 upper=0 effort=0.0 velocity=0.0
- joint link5-link6: limit lower=-3.140 upper=3.140 effort=0.0 velocity=0.0 -> lower=-1.70 upper=3.140 effort=0.0 velocity=0.0; origin xyz=0.0022 0 0.0045 rpy=0 0 0.0 -> xyz=0.0022 0 0.005 rpy=0 0 0.0
